Commit message: feat: minimal run

File: urdf/arduino_actuator_control.xacro (robot description, xacro)
@@ -15,5 +15,5 @@
       <origin xyz="0 0 0" rpy="0 0 0" />
       <geometry>
-        <box size="0.4 0.2 0.1" />
+        <box size="0.4 0.4 0.1" />
       </geometry>
     </collision>
@@ -21,5 +21,5 @@
       <origin xyz="0 0 0" rpy="0 0 0" />
       <geometry>
-        <box size="0.4 0.2 0.1" />
+        <box size="0.4 0.4 0.1" />
       </geometry>
       <material name="blue" />
@@ -30,5 +30,5 @@
       <origin xyz="0 0 0" rpy="0 0 0" />
       <geometry>
-        <box size="0.2 0.2 0.1" />
+        <box size="0.4 0.1 0.1" />
       </geometry>
     </collision>
@@ -36,5 +36,5 @@
       <origin xyz="0 0 0" rpy="0 0 0" />
       <geometry>
-        <box size="0.2 0.2 0.1" />
+        <box size="0.4 0.1 0.1" />
       </geometry>
       <material name="blue" />
@@ -50,5 +50,5 @@
     <parent link="base" />
     <child link="rotor" />
-    <origin xyz="0 0 0" rpy="0 0 0" />
+    <origin xyz="0.25 0 0" rpy="0 1.57 0" />
     <axis xyz="0 1 0" />
     <dynamics damping="0.7" />
@@ -57,7 +57,7 @@
     <hardware>
       <plugin>robot_control_system/ArduinoActuatorInterface</plugin>
-      <param name="example_param_hw_start_duration_sec">0</param>
-      <param name="example_param_hw_stop_duration_sec">3.0</param>
-      <param name="example_param_hw_slowdown">100</param>
+      <param name="hw_start_duration_sec">0</param>
+      <param name="hw_stop_duration_sec">3.0</param>
+      <param name="hw_slowdown">100</param>
     </hardware>
     <joint name="joint2">
