Commit message: feat: updated orientation for rotor

File: robot_control_system/urdf/arduino_actuator_control.xacro (robot description, xacro)
@@ -51,5 +51,5 @@
     <child link="rotor" />
     <origin xyz="0.25 0 0" rpy="0 1.57 0" />
-    <axis xyz="0 1 0" />
+    <axis xyz="0 0 1" />
     <dynamics damping="0.7" />
   </joint>
